File: design/DRV8301.kicad_sch (KiCad schematic)
At the start: 7 parts

Commit message: updates to BLDC
Parts:
- added C1, C2, C3: 100n, symbol Device:C_Small
- added C? (x2): 4u7_100V, Capacitor_SMD:C_0603_1608Metric_Pad1.08x0.95mm_HandSolder, symbol Device:C_Small
- added C? (x5): 2u2, Capacitor_SMD:C_0603_1608Metric_Pad1.08x0.95mm_HandSolder, symbol Device:C_Small
- added C? (x2): 15n, Capacitor_SMD:C_0603_1608Metric_Pad1.08x0.95mm_HandSolder, symbol Device:C_Small
- added C? (x3): 220n, Capacitor_SMD:C_0603_1608Metric_Pad1.08x0.95mm_HandSolder, symbol Device:C_Small
- added C?: 22n, Capacitor_SMD:C_0603_1608Metric_Pad1.08x0.95mm_HandSolder, symbol Device:C_Small
- added C?: 100u, Capacitor_SMD:C_1210_3225Metric, symbol Device:C_Small
- added D?: PMEG6020ER, Diode_SMD:Nexperia_CFP3_SOD-123W, symbol Diode:PMEG6020ER
- added L?: 22u, symbol Device:L
- added R1, R3, R5: 39k 60v, symbol Device:R_Small
- added R2, R4, R6: 2k2, symbol Device:R_Small
- added R?: 10k, Resistor_SMD:R_0603_1608Metric_Pad0.98x0.95mm_HandSolder, symbol Device:R_Small
- added R?: 10K, Resistor_SMD:R_0603_1608Metric_Pad0.98x0.95mm_HandSolder, symbol Device:R_Small
- added U1: ~, symbol Regulator_Linear:TC2117-3.3VDBTR
- added U2, U3, U4: MC74VHC1GT66, symbol Analog_Switch:MC74VHC1GT66
- U?: footprint Package_DFN_QFN:Texas_S-PVQFN-N40_EP3.52x2.62mm -> (none)
Connections:
- net +5V: now also C?.1, C?.1, L?.2, U1.3 (VI)
- net GND: now also U?.28 (AGND), U?.30 (SP2), U?.31 (SN2), U?.32 (SP1), U?.33 (SN1), C?.1, C?.1, C?.1, C?.1, C?.1, C?.2, C?.2, C?.2, C?.2, D?.2 (A), R2.2, R4.2, R6.2, R?.1, R?.2, U1.1 (GND), U2.2 (IO_YA), U2.3 (GND), U3.2 (IO_YA), U3.3 (GND), U4.2 (IO_YA), U4.3 (GND)
- net SDO: now reaches U?.10 (SDO)
- net SCLK: now reaches U?.11 (SCLK)
- net at U?.13 (GVDD): now also C?.2, C?.2
- net at U?.14 (CP1): now also C?.1
- net at U?.15 (CP2): now also C?.2
- net EN_GATE: now reaches U?.16 (EN_GATE)
- net EN_GATE: now also R?.2
- net INH_A: now reaches U?.17 (INH_A)
- net INL_A: now reaches U?.18 (INL_A)
- net INH_B: now reaches U?.19 (INH_B)
- net INL_B: now reaches U?.20 (INL_B)
- net INH_C: now reaches U?.21 (INH_C)
- net INL_C: now reaches U?.22 (INL_C)
- net at U?.23 (DVDD): now also C?.2
- net at U?.24 (REF): now also U?.27 (AVDD), C?.2
- net SUPPLY: now reaches U?.29 (PVDD1)
- net SUPPLY: now also U?.53 (PVDD2), U?.54 (PVDD2), C?.1, C?.1
- net SL_C: now reaches U?.34 (SL_C)
- net GL_C: now reaches U?.35 (GL_C)
- net SH_C: now reaches U?.36 (SH_C)
- net SH_C: now also C?.1, R5.2
- net GH_C: now reaches U?.37 (GH_C)
- net at U?.38 (BST_C): now also C?.2
- net SL_B: now reaches U?.39 (SL_B)
- net GL_B: now reaches U?.40 (GL_B)
- net SH_B: now reaches U?.41 (SH_B)
- net SH_B: now also C?.1, R3.2
- net GH_B: now reaches U?.42 (GH_B)
- net at U?.43 (BST_B): now also C?.2
- net SL_A: now reaches U?.44 (SL_A)
- net GL_A: now reaches U?.45 (GL_A)
- net SH_A: now reaches U?.46 (SH_A)
- net SH_A: now also C?.1, R1.2
- net GH_A: now reaches U?.47 (GH_A)
- net at U?.48 (BST_A): now also C?.2
- net +3.3V: now reaches U?.49 (VDD_SPI)
- net +3.3V: now also U1.2 (VO), U2.5 (VCC), U3.5 (VCC), U4.5 (VCC)
- net at U?.50 (PH): now also U?.51 (PH), C?.1, D?.1 (K), L?.1
- net at U?.52 (BST_BK): now also C?.2
- net EN_BUCK: now reaches U?.55 (EN_BUCK)
- net at U?.56 (SS_TR): now also C?.2
- net FAULT: now reaches U?.6 (nFAULT)
- net at U?.7 (DTC): now also R?.1
- net CS: now reaches U?.8 (nSCS)
- net SDI: now reaches U?.9 (SDI)
- new net: C3.2, U4.1 (IO_XA)
- new net: C2.2, U3.1 (IO_XA)
- new net: C1.2, U2.1 (IO_XA)
- new net SENS_A: C1.1, R1.1, R2.1
- new net SENS_B: C2.1, R3.1, R4.1
- new net SENS_C: C3.1, R5.1, R6.1
- no-connect marks 0 -> 5
Other:
- note added: "I had the genius idea to use the old BOM for the v4 to get the diode and a few other components"
- note added: "Place close to IC, internal VRef"

Commit message: more BLDC updates
Parts:
- added C4, C5: 2.2u, symbol Device:C_Small
- added C6: 100u, symbol Device:C_Polarized
- added D1: SMAJ5.0A, Diode_SMD:D_SMA, symbol Diode:SMAJ5.0A
- added Q2: Q_NMOS_GSD, symbol Device:Q_NMOS_GSD
- added R7: 2.2k, Resistor_SMD:R_0603_1608Metric_Pad0.98x0.95mm_HandSolder, symbol Device:R_Small
- added R8: 39k, Resistor_SMD:R_0603_1608Metric_Pad0.98x0.95mm_HandSolder, symbol Device:R_Small
Connections:
- net +3.3V: now also C5.1, C6.1
- net +5V: now also C4.1, D1.1 (A1), Q2.1 (G)
- net GND: now also C4.2, C5.2, C6.2, D1.2 (A2), R7.1
- net SUPPLY: now also R8.2
- new net: Q2.3 (D), R8.1
- new net SENS_SUPPLY: Q2.2 (S), R7.2
Other:
- moved on the sheet: U1
