File: design/DRV8301.kicad_sch (KiCad schematic)
At the start: 45 parts, among them Q2 Q_NMOS_GSD, U2 SN74LVC1G66DCKR, U3 SN74LVC1G66DCKR, U4 SN74LVC1G66DCKR

Commit message: finalised, ish, will have claude review
Parts:
- U2, U3, U4: value SN74LVC1G66DCKR -> MC74VHC1GT66; footprint Package_TO_SOT_SMD:SOT-353_SC-70-5 -> (none); symbol 74xGxx:74LVC1G66 -> Analog_Switch:MC74VHC1GT66
Connections:
- net +3.3V: now also U2.5 (VCC), U3.5 (VCC), U4.5 (VCC)
- net GND: now also U2.2 (IO_YA), U2.3 (GND), U3.2 (IO_YA), U3.3 (GND), U4.2 (IO_YA), U4.3 (GND)
- net SENS_FILTERED: now also U2.4 (ON_OFF), U3.4 (ON_OFF), U4.4 (ON_OFF)
- net at C3.2: now also U4.1 (IO_XA)
- net at C1.2: now also U2.1 (IO_XA)
- net at C2.2: now also U3.1 (IO_XA)
Changed lines of the file:
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@@
 	)
 	(symbol
-		(lib_id "74xGxx:74LVC1G66")
+		(lib_id "Analog_Switch:MC74VHC1GT66")
 		(at 118.745 174.625 0)
 		(unit 1)
@@
 			)
 		)
-		(property "Value" "SN74LVC1G66DCKR"
+		(property "Value" "MC74VHC1GT66"
 			(at 109.22 171.45 0)
 			(effects
@@
 			)
 		)
-		(property "Footprint" "Package_TO_SOT_SMD:SOT-353_SC-70-5"
+		(property "Footprint" ""
 			(at 109.855 172.085 0)
 			(effects
@@
 	)
 	(symbol
-		(lib_id "74xGxx:74LVC1G66")
+		(lib_id "Analog_Switch:MC74VHC1GT66")
 		(at 160.655 174.625 0)
 		(unit 1)
@@
 			)
 		)
-		(property "Value" "SN74LVC1G66DCKR"
+		(property "Value" "MC74VHC1GT66"
 			(at 151.13 171.45 0)
 			(effects
@@
 			)
 		)
-		(property "Footprint" "Package_TO_SOT_SMD:SOT-353_SC-70-5"
+		(property "Footprint" ""
 			(at 151.765 172.085 0)
 			(effects
@@
 	)
 	(symbol
-		(lib_id "74xGxx:74LVC1G66")
+		(lib_id "Analog_Switch:MC74VHC1GT66")
 		(at 73.025 174.625 0)
 		(unit 1)
@@
 			)
 		)
-		(property "Value" "SN74LVC1G66DCKR"
+		(property "Value" "MC74VHC1GT66"
 			(at 63.5 171.45 0)
 			(effects
@@
 			)
 		)
-		(property "Footprint" "Package_TO_SOT_SMD:SOT-353_SC-70-5"
+		(property "Footprint" ""
 			(at 64.135 172.085 0)
 			(effects
