File: design/DRV8301.kicad_sch (KiCad schematic)
At the start: 45 parts, among them Q2 Q_NMOS_GSD, U2 MC74VHC1GT66, U3 MC74VHC1GT66, U4 MC74VHC1GT66

Commit message: Sheet 3 (DRV8301.kicad_sch): assign footprints, update parts, fix issues
MC-002 partial: BST_A D? PMEG6020ER → DSS210 (100V, SOD-123F). BST_B/C still need placement in KiCad.
MC-004 resolved: DRV8301 U? footprint set to Texas_HTSSOP-56_6.1x9.7mm_P0.65mm.
MC-006 resolved: TC2117 U1 Value set (was ~), Footprint SOT-223-3_TabPin2.
MC-008 resolved: Q2 SENS_SUPPLY assigned BSS138 / SOT-23.
MC-014 partial: U2/U3/U4 Value → SN74LVC1G66DCKR, Footprint → SOT-353_SC-70-5 (lib_id kept compatible).

Blank footprints filled in: C1/C2/C3 (100n 0603), C4/C5 (2.2u 0805), C6 (100u elec), R1-R6 (0603), L? (1008).

Co-Authored-By: Claude Sonnet 4.6 <noreply@anthropic.com>
Parts:
- C1, C2, C3: footprint (none) -> Capacitor_SMD:C_0603_1608Metric_Pad1.08x0.95mm_HandSolder
- C4, C5: footprint (none) -> Capacitor_SMD:C_0805_2012Metric_Pad1.18x1.45mm_HandSolder
- C6: footprint (none) -> Capacitor_SMD:CP_Elec_10x10.5
- D?: value PMEG6020ER -> DSS210; footprint Diode_SMD:Nexperia_CFP3_SOD-123W -> Diode_SMD:D_SOD-123F
- L?: footprint (none) -> Inductor_SMD:L_1008_2520Metric
- Q2: value Q_NMOS_GSD -> BSS138; footprint (none) -> Package_TO_SOT_SMD:SOT-23
- R1, R2, R3, R4, R5, R6: footprint (none) -> Resistor_SMD:R_0603_1608Metric_Pad0.98x0.95mm_HandSolder
- U1: value ~ -> TC2117-3.3VDBTR; footprint (none) -> Package_TO_SOT_SMD:SOT-223-3_TabPin2
- U2, U3, U4: value MC74VHC1GT66 -> SN74LVC1G66DCKR; footprint (none) -> Package_TO_SOT_SMD:SOT-353_SC-70-5
- U?: footprint (none) -> Package_SO:Texas_HTSSOP-56_6.1x9.7mm_P0.65mm
Changed lines of the file:
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@@
 			)
 		)
-		(property "Footprint" ""
+		(property "Footprint" "Capacitor_SMD:CP_Elec_10x10.5"
 			(at 247.3452 148.59 0)
 			(effects
@@
 			)
 		)
-		(property "Footprint" ""
+		(property "Footprint" "Capacitor_SMD:C_0603_1608Metric_Pad1.08x0.95mm_HandSolder"
 			(at 152.4 165.1 0)
 			(effects
@@
 			)
 		)
-		(property "Footprint" ""
+		(property "Footprint" "Resistor_SMD:R_0603_1608Metric_Pad0.98x0.95mm_HandSolder"
 			(at 109.855 157.48 0)
 			(effects
@@
 			)
 		)
-		(property "Footprint" ""
+		(property "Footprint" "Inductor_SMD:L_1008_2520Metric"
 			(at 192.532 71.12 0)
 			(effects
@@
 			)
 		)
-		(property "Footprint" ""
+		(property "Footprint" "Resistor_SMD:R_0603_1608Metric_Pad0.98x0.95mm_HandSolder"
 			(at 64.135 154.305 0)
 			(effects
@@
 			)
 		)
-		(property "Value" "MC74VHC1GT66"
+		(property "Value" "SN74LVC1G66DCKR"
 			(at 109.22 171.45 0)
 			(effects
@@
 			)
 		)
-		(property "Footprint" ""
+		(property "Footprint" "Package_TO_SOT_SMD:SOT-353_SC-70-5"
 			(at 109.855 172.085 0)
 			(effects
@@
 			)
 		)
-		(property "Footprint" ""
+		(property "Footprint" "Resistor_SMD:R_0603_1608Metric_Pad0.98x0.95mm_HandSolder"
 			(at 151.765 157.48 0)
 			(effects
@@
 			)
 		)
-		(property "Value" "MC74VHC1GT66"
+		(property "Value" "SN74LVC1G66DCKR"
 			(at 151.13 171.45 0)
 			(effects
@@
 			)
 		)
-		(property "Footprint" ""
+		(property "Footprint" "Package_TO_SOT_SMD:SOT-353_SC-70-5"
 			(at 151.765 172.085 0)
 			(effects
@@
 			)
 		)
-		(property "Footprint" ""
+		(property "Footprint" "Capacitor_SMD:C_0805_2012Metric_Pad1.18x1.45mm_HandSolder"
 			(at 235.585 144.145 0)
 			(effects
@@
 			)
 		)
-		(property "Footprint" ""
+		(property "Footprint" "Capacitor_SMD:C_0603_1608Metric_Pad1.08x0.95mm_HandSolder"
 			(at 64.77 165.1 0)
 			(effects
@@
 			)
 		)
-		(property "Value" "~"
+		(property "Value" "TC2117-3.3VDBTR"
 			(at 222.25 138.43 0)
 			(effects
@@
 			)
 		)
-		(property "Footprint" ""
+		(property "Footprint" "Package_TO_SOT_SMD:SOT-223-3_TabPin2"
 			(at 222.25 139.7 0)
 			(effects
@@
 			)
 		)
-		(property "Value" "Q_NMOS_GSD"
+		(property "Value" "BSS138"
 			(at 248.285 99.6949 0)
 			(effects
@@
 			)
 		)
-		(property "Footprint" ""
+		(property "Footprint" "Package_TO_SOT_SMD:SOT-23"
 			(at 247.65 95.885 0)
 			(effects
@@
 			)
 		)
-		(property "Footprint" ""
+		(property "Footprint" "Package_SO:Texas_HTSSOP-56_6.1x9.7mm_P0.65mm"
 			(at 146.05 137.16 0)
 			(effects
@@
 			)
 		)
-		(property "Value" "PMEG6020ER"
+		(property "Value" "DSS210"
 			(at 183.896 71.374 0)
 			(effects
@@
 			)
 		)
-		(property "Footprint" "Diode_SMD:Nexperia_CFP3_SOD-123W"
+		(property "Footprint" "Diode_SMD:D_SOD-123F"
 			(at 182.245 75.946 0)
 			(effects
@@
 			)
 		)
-		(property "Value" "MC74VHC1GT66"
+		(property "Value" "SN74LVC1G66DCKR"
 			(at 63.5 171.45 0)
 			(effects
@@
 			)
 		)
-		(property "Footprint" ""
+		(property "Footprint" "Package_TO_SOT_SMD:SOT-353_SC-70-5"
 			(at 64.135 172.085 0)
 			(effects
@@
 			)
 		)
-		(property "Footprint" ""
+		(property "Footprint" "Resistor_SMD:R_0603_1608Metric_Pad0.98x0.95mm_HandSolder"
 			(at 151.765 154.305 0)
 			(effects
@@
 			)
 		)
-		(property "Footprint" ""
+		(property "Footprint" "Resistor_SMD:R_0603_1608Metric_Pad0.98x0.95mm_HandSolder"
 			(at 109.855 154.305 0)
 			(effects
@@
 			)
 		)
-		(property "Footprint" ""
+		(property "Footprint" "Capacitor_SMD:C_0805_2012Metric_Pad1.18x1.45mm_HandSolder"
 			(at 201.295 144.145 0)
 			(effects
@@
 			)
 		)
-		(property "Footprint" ""
+		(property "Footprint" "Resistor_SMD:R_0603_1608Metric_Pad0.98x0.95mm_HandSolder"
 			(at 64.135 157.48 0)
 			(effects
@@
 			)
 		)
-		(property "Footprint" ""
+		(property "Footprint" "Capacitor_SMD:C_0603_1608Metric_Pad1.08x0.95mm_HandSolder"
 			(at 110.49 165.1 0)
 			(effects

Commit message: L? inductor: assign SMNR4020-22UH (LCSC C135264)
22µH ±20%, 1.05A Isat, 455mΩ DCR, 4×4×2mm SMD.
Footprint corrected from L_1008_2520Metric → L_4040_Coilcraft_DO3316.
LCSC property added to schematic symbol.
BOM.md updated with selected part.

Co-Authored-By: Claude Sonnet 4.6 <noreply@anthropic.com>
Parts:
- L1: renamed from L?; footprint Inductor_SMD:L_1008_2520Metric -> Inductor_SMD:L_4040_Coilcraft_DO3316; LCSC (none) -> C135264
- gave numbers to parts that had none: 24
- renumbered C4 to C33, C5 to C34, C6 to C35, C1 to C36, C2 to C37, C3 to C38, D1 to D10, Q2 to Q1, R8 to R25, R7 to R27, R1 to R28, R3 to R29, R5 to R30, R2 to R31, R4 to R32, R6 to R33, U1 to U4, U2 to U5, U3 to U6, U4 to U7

Commit message: All sheets: add LCSC part numbers to 136 components
Populated LCSC Cxxxxxx properties on every assigned component across all
6 sheets (SBS_hw, MCU, DRV8301, CAN, BMI160, Power). Remaining ~19
components (15nF/120pF 0603 caps, 2.2µF 0805, 100µF electrolytic/1210,
1k PTC, 1.27mm SWD header, solder jumper, single-pin placeholders) have
no confirmed LCSC number and are left unpopulated.

Co-Authored-By: Claude Sonnet 4.6 <noreply@anthropic.com>
Claude-Session: https://claude.ai/code/session_01DS1NowMbUxuJRBVhV127qS
Parts:
- C17: LCSC (none) -> C1631
- C20, C32: LCSC (none) -> C338088
- C22, C25, C28, C30, C31: LCSC (none) -> C23630
- C24, C27, C29: LCSC (none) -> C21120
- C26: LCSC (none) -> C21122
- C36, C37, C38: LCSC (none) -> C14663
- D10: LCSC (none) -> C87074
- D9: LCSC (none) -> C511868
- Q1: LCSC (none) -> C112739
- R20: LCSC (none) -> C22978
- R21: LCSC (none) -> C22961
- R22: LCSC (none) -> C25810
- R23: LCSC (none) -> C22809
- R24, R26: LCSC (none) -> C25804
- R25, R28, R29, R30: LCSC (none) -> C23153
- R27, R31, R32, R33: LCSC (none) -> C4190
- U3: LCSC (none) -> C98969
- U4: LCSC (none) -> C98655
- U5, U6, U7: LCSC (none) -> C113518
