File: design/DRV8301.kicad_sch (KiCad schematic)
At the start: 45 parts, among them Q1 BSS138, U3 3_Phase_BLDC_Driver_56_Pin_HT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, U4 TC2117-3.3VDBTR, U5 SN74LVC1G66DCKR, U6 SN74LVC1G66DCKR, U7 SN74LVC1G66DCKR

Commit message: schematic basicaly done. mechanical design fleshed out
Parts:
- Q1: LCSC C112739 -> C52895
Changed lines of the file:
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@@
 			)
 		)
-		(property "LCSC" "C112739"
+		(property "LCSC" "C52895"
 			(at 0 0 0)
 			(effects
