File: design/Power.kicad_sch (KiCad schematic)
At the start: 8 parts, among them Q1 IRF7749L1TRPBF, Q3 IRF7749L1TRPBF, U5 AD8418

Commit message: finalised, ish, will have claude review
Parts:
- added C10, C11, C13, C14, C8, C9: CGA6M3X7S2A475KT0Y3S, Capacitor_SMD:C_1210_3225Metric_Pad1.33x2.70mm_HandSolder, symbol Device:C_Small
- added C12, C15: 2u2, Capacitor_SMD:C_0603_1608Metric_Pad1.08x0.95mm_HandSolder, symbol Device:C_Small
- added C16, C18, C20: 15n, symbol Device:C_Small
- added C17, C19, C21: 1n, symbol Device:C_Small
- added C22: 2u2, symbol Device:C_Small
- added J1: SUPPLY, symbol Connector:Screw_Terminal_01x01
- added J2: GND, symbol Connector:Screw_Terminal_01x01
- added PH_B, PH_C: ~, symbol Connector:Solder_Pad
- added Q4, Q5, Q6, Q7: IRF7749L1TRPBF, Package_DirectFET:DirectFET_L8, symbol Transistor_FET:IRF7748L1
- added R12, R14, R15, R17: 4.7R, Resistor_SMD:R_0402_1005Metric, symbol Device:R_Small
- added R13, R16: 0.0005, symbol Device:R_Small
- added R18, R19, R20: 1k, symbol Device:R_Small
- added R21: 10k, symbol Device:R_Small
- added TH1: 10k, symbol Device:Thermistor_NTC
- added U10, U8, U9: MC74VHC1GT66, symbol Analog_Switch:MC74VHC1GT66
- added U6, U7: AD8418, symbol Amplifier_Current:AD8418
- C7: value 100n -> 2u2
Connections:
- net C_A: now also R18.2
- net GND: now also Q3.3 (S), C10.2, C11.2, C12.1, C13.2, C14.2, C15.1, C16.2, C17.2, C18.2, C19.2, C20.2, C21.2, C22.2, C8.2, C9.2, J2.1 (Pin_1), Q5.3 (S), Q7.3 (S), R21.2, U10.3 (GND), U6.2 (GND), U6.3 (REF2), U7.2 (GND), U7.3 (REF2), U8.3 (GND), U9.3 (GND)
- net SH_A: now reaches Q1.3 (S), R9.2, U5.1 (IN-)
- net SH_A: now also Q3.1 (D)
- net +3.3V: now reaches C7.2, U5.6 (VS), U5.7 (REF1)
- net +3.3V: now also C12.2, C15.2, TH1.1, U10.5 (VCC), U6.6 (VS), U6.7 (REF1), U7.6 (VS), U7.7 (REF1), U8.5 (VCC), U9.5 (VCC)
- net SUPPLY: now reaches Q1.1 (D)
- net SUPPLY: now also C10.1, C11.1, C13.1, C14.1, C8.1, C9.1, J1.1 (Pin_1), Q4.1 (D), Q6.1 (D)
- net GL_A: now reaches R11.1
- new net: Q6.3 (S), Q7.1 (D), R16.2, U7.1 (IN-)
- new net: Q7.2 (G), R17.2
- new net: Q5.2 (G), R14.2
- new net: C16.1, U8.2 (IO_YA)
- new net: C20.1, U10.2 (IO_YA)
- new net: C18.1, U9.2 (IO_YA)
- new net: PH_B.1, R13.1, U6.8 (IN+)
- new net: Q4.2 (G), R12.2
- new net: Q6.2 (G), R15.2
- new net: PH_C.1, R16.1, U7.8 (IN+)
- new net CURR_A: C17.1, R18.1, U8.1 (IO_XA)
- new net CURR_B: C19.1, R19.1, U9.1 (IO_XA)
- new net CURR_C: C21.1, R20.1, U10.1 (IO_XA)
- new net CURR_FILTER: U10.4 (ON_OFF), U8.4 (ON_OFF), U9.4 (ON_OFF)
- new net C_B: R19.2, U6.5 (OUT)
- new net C_C: R20.2, U7.5 (OUT)
- new net GH_B: R12.1
- new net GH_C: R15.1
- new net GL_B: R14.1
- new net GL_C: R17.1
- new net SH_B: Q4.3 (S), Q5.1 (D), R13.2, U6.1 (IN-)
- new net TEMP: C22.1, R21.1, TH1.2
Other:
- note added: "1/(2*pi*R*C) = 159 kHz or 10Khz when we parallel the 15n"
- note added: "4u7 100V"
- note added: "NTC"
- note added: "does it make sense to have 6 of these capacitors in parallel?"
- moved on the sheet: C7, PH_A, Q1, Q3, R10, R11, R9, U5
