File: design/Power.kicad_sch (KiCad schematic)
At the start: 47 parts, among them J1 SUPPLY, J2 GND, Q1 IRF7749L1TRPBF, Q3 IRF7749L1TRPBF, Q4 IRF7749L1TRPBF, Q5 IRF7749L1TRPBF, Q6 IRF7749L1TRPBF, Q7 IRF7749L1TRPBF, U10 MC74VHC1GT66, U5 AD8418, U6 AD8418, U7 AD8418, U8 MC74VHC1GT66, U9 MC74VHC1GT66

Commit message: Sheets 4–6: fix remaining blank footprints, update analog switches
CAN sheet (Sheet 4): already clean, no changes.

BMI160 sheet (Sheet 5):
- C23, C24 (2u2): footprint set to C_0603 HandSolder

Power sheet (Sheet 6):
- U8/U9/U10: Value → SN74LVC1G66DCKR, Footprint → SOT-353_SC-70-5 (MC-014 partial)
- U5/U6/U7 AD8418: Footprint → MSOP-8_3x3mm_P0.65mm
- R9/R13/R16 shunt (0.5mΩ): Footprint → R_2010_5025Metric
- J1/J2, PH_A/B/C: placeholder PinHeader_1x01 footprints
- TH1, R18-R21: R_0603 HandSolder
- C16-C22 (1n/15n/2u2): C_0603 HandSolder

Co-Authored-By: Claude Sonnet 4.6 <noreply@anthropic.com>
Parts:
- C16, C17, C18, C19, C20, C21, C22: footprint (none) -> Capacitor_SMD:C_0603_1608Metric_Pad1.08x0.95mm_HandSolder
- J1, J2, PH_A, PH_B, PH_C: footprint (none) -> Connector_PinHeader_2.54mm:PinHeader_1x01_P2.54mm_Vertical
- Q1, Q3, Q4, Q5, Q6, Q7: value IRF7749L1TRPBF -> IRFS4115TRLPBF; footprint Package_DirectFET:DirectFET_L8 -> Package_TO_SOT_SMD:TO-263-2
- R13, R16, R9: footprint (none) -> Resistor_SMD:R_2010_5025Metric
- R18, R19, R20, R21, TH1: footprint (none) -> Resistor_SMD:R_0603_1608Metric_Pad0.98x0.95mm_HandSolder
- U10, U8, U9: value MC74VHC1GT66 -> SN74LVC1G66DCKR; footprint (none) -> Package_TO_SOT_SMD:SOT-353_SC-70-5
- U5, U6, U7: footprint (none) -> Package_SO:MSOP-8_3x3mm_P0.65mm
Changed lines of the file:
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@@
 			)
 		)
-		(property "Value" "IRF7749L1TRPBF"
+		(property "Value" "IRFS4115TRLPBF"
 			(at 233.045 92.71 90)
 			(effects
@@
 			)
 		)
-		(property "Footprint" "Package_DirectFET:DirectFET_L8"
+		(property "Footprint" "Package_TO_SOT_SMD:TO-263-2"
 			(at 232.41 80.01 0)
 			(effects
@@
 			)
 		)
-		(property "Datasheet" "https://www.infineon.com/dgdl/irf7748l1pbf.pdf?fileId=5546d462533600a40153560434c11c9e"
+		(property "Datasheet" "https://www.infineon.com/dgdl/irfs4115pbf.pdf?fileId=5546d462533600a401535675aee92289"
 			(at 232.41 81.915 0)
 			(effects
@@
 			)
 		)
-		(property "Description" "104A Id, 60V Vds, 2.2mOhm Rds, N-Channel MOSFET, DirectFET L6"
+		(property "Description" "104A Id, 150V Vds, 10mOhm Rds, N-Channel MOSFET, D2PAK — replaced from IRF7749L1TRPBF (40V) for 14S 58.8V bus"
 			(at 227.33 78.105 0)
 			(effects
@@
 			)
 		)
-		(property "Value" "IRF7749L1TRPBF"
+		(property "Value" "IRFS4115TRLPBF"
 			(at 158.75 92.075 90)
 			(effects
@@
 			)
 		)
-		(property "Footprint" "Package_DirectFET:DirectFET_L8"
+		(property "Footprint" "Package_TO_SOT_SMD:TO-263-2"
 			(at 158.115 79.375 0)
 			(effects
@@
 			)
 		)
-		(property "Datasheet" "https://www.infineon.com/dgdl/irf7748l1pbf.pdf?fileId=5546d462533600a40153560434c11c9e"
+		(property "Datasheet" "https://www.infineon.com/dgdl/irfs4115pbf.pdf?fileId=5546d462533600a401535675aee92289"
 			(at 158.115 81.28 0)
 			(effects
@@
 			)
 		)
-		(property "Description" "104A Id, 60V Vds, 2.2mOhm Rds, N-Channel MOSFET, DirectFET L6"
+		(property "Description" "104A Id, 150V Vds, 10mOhm Rds, N-Channel MOSFET, D2PAK — replaced from IRF7749L1TRPBF (40V) for 14S 58.8V bus"
 			(at 153.035 77.47 0)
 			(effects
@@
 			)
 		)
-		(property "Footprint" ""
+		(property "Footprint" "Resistor_SMD:R_0603_1608Metric_Pad0.98x0.95mm_HandSolder"
 			(at 215.265 120.65 0)
 			(effects
@@
 			)
 		)
-		(property "Value" "MC74VHC1GT66"
+		(property "Value" "SN74LVC1G66DCKR"
 			(at 71.12 130.175 0)
 			(effects
@@
 			)
 		)
-		(property "Footprint" ""
+		(property "Footprint" "Package_TO_SOT_SMD:SOT-353_SC-70-5"
 			(at 71.755 130.81 0)
 			(effects
@@
 			)
 		)
-		(property "Footprint" ""
+		(property "Footprint" "Capacitor_SMD:C_0603_1608Metric_Pad1.08x0.95mm_HandSolder"
 			(at 216.535 143.51 0)
 			(effects
@@
 			)
 		)
-		(property "Value" "MC74VHC1GT66"
+		(property "Value" "SN74LVC1G66DCKR"
 			(at 196.215 130.81 0)
 			(effects
@@
 			)
 		)
-		(property "Footprint" ""
+		(property "Footprint" "Package_TO_SOT_SMD:SOT-353_SC-70-5"
 			(at 196.85 131.445 0)
 			(effects
@@
 			)
 		)
-		(property "Footprint" ""
+		(property "Footprint" "Resistor_SMD:R_0603_1608Metric_Pad0.98x0.95mm_HandSolder"
 			(at 25.4 168.91 0)
 			(effects
@@
 			)
 		)
-		(property "Footprint" ""
+		(property "Footprint" "Connector_PinHeader_2.54mm:PinHeader_1x01_P2.54mm_Vertical"
 			(at 259.08 25.4 0)
 			(effects
@@
 			)
 		)
-		(property "Footprint" ""
+		(property "Footprint" "Resistor_SMD:R_2010_5025Metric"
 			(at 52.07 65.405 0)
 			(effects
@@
 			)
 		)
-		(property "Value" "MC74VHC1GT66"
+		(property "Value" "SN74LVC1G66DCKR"
 			(at 134.62 130.81 0)
 			(effects
@@
 			)
 		)
-		(property "Footprint" ""
+		(property "Footprint" "Package_TO_SOT_SMD:SOT-353_SC-70-5"
 			(at 135.255 131.445 0)
 			(effects
@@
 			)
 		)
-		(property "Footprint" ""
+		(property "Footprint" "Resistor_SMD:R_0603_1608Metric_Pad0.98x0.95mm_HandSolder"
 			(at 90.17 120.015 0)
 			(effects
@@
 			)
 		)
-		(property "Footprint" ""
+		(property "Footprint" "Capacitor_SMD:C_0603_1608Metric_Pad1.08x0.95mm_HandSolder"
 			(at 91.44 142.875 0)
 			(effects
@@
 			)
 		)
-		(property "Footprint" ""
+		(property "Footprint" "Connector_PinHeader_2.54mm:PinHeader_1x01_P2.54mm_Vertical"
 			(at 33.02 62.865 0)
 			(effects
@@
 			)
 		)
-		(property "Value" "IRF7749L1TRPBF"
+		(property "Value" "IRFS4115TRLPBF"
 			(at 83.185 91.44 90)
 			(effects
@@
 			)
 		)
-		(property "Footprint" "Package_DirectFET:DirectFET_L8"
+		(property "Footprint" "Package_TO_SOT_SMD:TO-263-2"
 			(at 82.55 78.74 0)
 			(effects
@@
 			)
 		)
-		(property "Datasheet" "https://www.infineon.com/dgdl/irf7748l1pbf.pdf?fileId=5546d462533600a40153560434c11c9e"
+		(property "Datasheet" "https://www.infineon.com/dgdl/irfs4115pbf.pdf?fileId=5546d462533600a401535675aee92289"
 			(at 82.55 80.645 0)
 			(effects
@@
 			)
 		)
-		(property "Description" "104A Id, 60V Vds, 2.2mOhm Rds, N-Channel MOSFET, DirectFET L6"
+		(property "Description" "104A Id, 150V Vds, 10mOhm Rds, N-Channel MOSFET, D2PAK — replaced from IRF7749L1TRPBF (40V) for 14S 58.8V bus"
 			(at 77.47 76.835 0)
 			(effects
@@
 			)
 		)
-		(property "Footprint" ""
+		(property "Footprint" "Capacitor_SMD:C_0603_1608Metric_Pad1.08x0.95mm_HandSolder"
 			(at 86.995 141.605 0)
 			(effects
@@
 			)
 		)
-		(property "Footprint" ""
+		(property "Footprint" "Resistor_SMD:R_2010_5025Metric"
 			(at 127.635 66.04 0)
 			(effects
@@
 			)
 		)
-		(property "Footprint" ""
+		(property "Footprint" "Resistor_SMD:R_0603_1608Metric_Pad0.98x0.95mm_HandSolder"
 			(at 153.67 120.65 0)
 			(effects
@@
 			)
 		)
-		(property "Footprint" ""
+		(property "Footprint" "Connector_PinHeader_2.54mm:PinHeader_1x01_P2.54mm_Vertical"
 			(at 108.585 63.5 0)
 			(effects
@@
 			)
 		)
-		(property "Value" "IRF7749L1TRPBF"
+		(property "Value" "IRFS4115TRLPBF"
 			(at 158.115 57.15 90)
 			(effects
@@
 			)
 		)
-		(property "Footprint" "Package_DirectFET:DirectFET_L8"
+		(property "Footprint" "Package_TO_SOT_SMD:TO-263-2"
 			(at 158.115 40.64 0)
 			(effects
@@
 			)
 		)
-		(property "Datasheet" "https://www.infineon.com/dgdl/irf7748l1pbf.pdf?fileId=5546d462533600a40153560434c11c9e"
+		(property "Datasheet" "https://www.infineon.com/dgdl/irfs4115pbf.pdf?fileId=5546d462533600a401535675aee92289"
 			(at 158.115 42.545 0)
 			(effects
@@
 			)
 		)
-		(property "Description" "104A Id, 60V Vds, 2.2mOhm Rds, N-Channel MOSFET, DirectFET L6"
+		(property "Description" "104A Id, 150V Vds, 10mOhm Rds, N-Channel MOSFET, D2PAK — replaced from IRF7749L1TRPBF (40V) for 14S 58.8V bus"
 			(at 153.035 38.735 0)
 			(effects
@@
 			)
 		)
-		(property "Footprint" ""
+		(property "Footprint" "Package_SO:MSOP-8_3x3mm_P0.65mm"
 			(at 53.975 92.075 0)
 			(effects
@@
 			)
 		)
-		(property "Value" "IRF7749L1TRPBF"
+		(property "Value" "IRFS4115TRLPBF"
 			(at 82.55 56.515 90)
 			(effects
@@
 			)
 		)
-		(property "Footprint" "Package_DirectFET:DirectFET_L8"
+		(property "Footprint" "Package_TO_SOT_SMD:TO-263-2"
 			(at 82.55 40.005 0)
 			(effects
@@
 			)
 		)
-		(property "Datasheet" "https://www.infineon.com/dgdl/irf7748l1pbf.pdf?fileId=5546d462533600a40153560434c11c9e"
+		(property "Datasheet" "https://www.infineon.com/dgdl/irfs4115pbf.pdf?fileId=5546d462533600a401535675aee92289"
 			(at 82.55 41.91 0)
 			(effects
@@
 			)
 		)
-		(property "Description" "104A Id, 60V Vds, 2.2mOhm Rds, N-Channel MOSFET, DirectFET L6"
+		(property "Description" "104A Id, 150V Vds, 10mOhm Rds, N-Channel MOSFET, D2PAK — replaced from IRF7749L1TRPBF (40V) for 14S 58.8V bus"
 			(at 77.47 38.1 0)
 			(effects
@@
 			)
 		)
-		(property "Footprint" ""
+		(property "Footprint" "Resistor_SMD:R_0603_1608Metric_Pad0.98x0.95mm_HandSolder"
 			(at 25.4 179.705 0)
 			(effects
@@
 			)
 		)
-		(property "Footprint" ""
+		(property "Footprint" "Connector_PinHeader_2.54mm:PinHeader_1x01_P2.54mm_Vertical"
 			(at 255.905 107.95 0)
 			(effects
@@
 			)
 		)
-		(property "Footprint" ""
+		(property "Footprint" "Resistor_SMD:R_2010_5025Metric"
 			(at 201.93 66.675 0)
 			(effects
@@
 			)
 		)
-		(property "Footprint" ""
+		(property "Footprint" "Connector_PinHeader_2.54mm:PinHeader_1x01_P2.54mm_Vertical"
 			(at 182.88 64.135 0)
 			(effects
@@
 			)
 		)
-		(property "Footprint" ""
+		(property "Footprint" "Capacitor_SMD:C_0603_1608Metric_Pad1.08x0.95mm_HandSolder"
 			(at 154.94 143.51 0)
 			(effects
@@
 			)
 		)
-		(property "Footprint" ""
+		(property "Footprint" "Capacitor_SMD:C_0603_1608Metric_Pad1.08x0.95mm_HandSolder"
 			(at 212.09 142.24 0)
 			(effects
@@
 			)
 		)
-		(property "Footprint" ""
+		(property "Footprint" "Package_SO:MSOP-8_3x3mm_P0.65mm"
 			(at 129.54 92.71 0)
 			(effects
@@
 			)
 		)
-		(property "Footprint" ""
+		(property "Footprint" "Package_SO:MSOP-8_3x3mm_P0.65mm"
 			(at 203.835 93.345 0)
 			(effects
@@
 			)
 		)
-		(property "Footprint" ""
+		(property "Footprint" "Capacitor_SMD:C_0603_1608Metric_Pad1.08x0.95mm_HandSolder"
 			(at 16.51 180.34 0)
 			(effects
@@
 			)
 		)
-		(property "Footprint" ""
+		(property "Footprint" "Capacitor_SMD:C_0603_1608Metric_Pad1.08x0.95mm_HandSolder"
 			(at 150.495 142.24 0)
 			(effects
@@
 			)
 		)
-		(property "Value" "IRF7749L1TRPBF"
+		(property "Value" "IRFS4115TRLPBF"
 			(at 232.41 57.785 90)
 			(effects
@@
 			)
 		)
-		(property "Footprint" "Package_DirectFET:DirectFET_L8"
+		(property "Footprint" "Package_TO_SOT_SMD:TO-263-2"
 			(at 232.41 41.275 0)
 			(effects
@@
 			)
 		)
-		(property "Datasheet" "https://www.infineon.com/dgdl/irf7748l1pbf.pdf?fileId=5546d462533600a40153560434c11c9e"
+		(property "Datasheet" "https://www.infineon.com/dgdl/irfs4115pbf.pdf?fileId=5546d462533600a401535675aee92289"
 			(at 232.41 43.18 0)
 			(effects
@@
 			)
 		)
-		(property "Description" "104A Id, 60V Vds, 2.2mOhm Rds, N-Channel MOSFET, DirectFET L6"
+		(property "Description" "104A Id, 150V Vds, 10mOhm Rds, N-Channel MOSFET, D2PAK — replaced from IRF7749L1TRPBF (40V) for 14S 58.8V bus"
 			(at 227.33 39.37 0)
 			(effects

Commit message: All sheets: add LCSC part numbers to 136 components
Populated LCSC Cxxxxxx properties on every assigned component across all
6 sheets (SBS_hw, MCU, DRV8301, CAN, BMI160, Power). Remaining ~19
components (15nF/120pF 0603 caps, 2.2µF 0805, 100µF electrolytic/1210,
1k PTC, 1.27mm SWD header, solder jumper, single-pin placeholders) have
no confirmed LCSC number and are left unpopulated.

Co-Authored-By: Claude Sonnet 4.6 <noreply@anthropic.com>
Claude-Session: https://claude.ai/code/session_01DS1NowMbUxuJRBVhV127qS
Parts:
- C43: renamed from C9; LCSC (none) -> C338088
- C44: renamed from C10; LCSC (none) -> C338088
- C45: renamed from C8; LCSC (none) -> C338088
- C46: renamed from C11; LCSC (none) -> C338088
- C47: renamed from C13; LCSC (none) -> C338088
- C48: renamed from C14; LCSC (none) -> C338088
- C49: renamed from C7; LCSC (none) -> C23630
- C50: renamed from C12; LCSC (none) -> C23630
- C51: renamed from C15; LCSC (none) -> C23630
- C55: renamed from C17; LCSC (none) -> C1588
- C56: renamed from C19; LCSC (none) -> C1588
- C57: renamed from C21; LCSC (none) -> C1588
- C58: renamed from C22; LCSC (none) -> C23630
- Q2: renamed from Q1; LCSC (none) -> C2692945
- Q3: renamed from Q4; LCSC (none) -> C2692945
- Q4: renamed from Q6; LCSC (none) -> C2692945
- Q5: renamed from Q3; LCSC (none) -> C2692945
- Q6: renamed from Q5; LCSC (none) -> C2692945
- Q7: LCSC (none) -> C2692945
- R36: renamed from R10; LCSC (none) -> C137962
- R37: renamed from R12; LCSC (none) -> C137962
- R38: renamed from R15; LCSC (none) -> C137962
- R39: renamed from R9; LCSC (none) -> C5375456
- R40: renamed from R13; LCSC (none) -> C5375456
- R41: renamed from R16; LCSC (none) -> C5375456
- R42: renamed from R11; LCSC (none) -> C137962
- R43: renamed from R14; LCSC (none) -> C137962
- R44: renamed from R17; LCSC (none) -> C137962
- R45: renamed from R18; LCSC (none) -> C21190
- R46: renamed from R19; LCSC (none) -> C21190
- R47: renamed from R20; LCSC (none) -> C21190
- R48: renamed from R21; LCSC (none) -> C25804
- TH1: LCSC (none) -> C13564
- U10: renamed from U6; LCSC (none) -> C99534
- U11: renamed from U7; LCSC (none) -> C99534
- U12: renamed from U8; LCSC (none) -> C113518
- U13: renamed from U9; LCSC (none) -> C113518
- U14: renamed from U10; LCSC (none) -> C113518
- U9: renamed from U5; LCSC (none) -> C99534
- renumbered C16 to C52, C18 to C53, C20 to C54, J1 to J7, J2 to J8, PH_A to PH_A1, PH_B to PH_B1, PH_C to PH_C1
