File: design/Power.kicad_sch (KiCad schematic)
At the start: 47 parts, among them J7 SUPPLY, J8 GND, Q2 IRFS4115TRLPBF, Q3 IRFS4115TRLPBF, Q4 IRFS4115TRLPBF, Q5 IRFS4115TRLPBF, Q6 IRFS4115TRLPBF, Q7 IRFS4115TRLPBF, U10 AD8418, U11 AD8418, U12 SN74LVC1G66DCKR, U13 SN74LVC1G66DCKR, U14 SN74LVC1G66DCKR, U9 AD8418

Commit message: schematic basicaly done. mechanical design fleshed out
Parts:
- Q2, Q3, Q4, Q5, Q6, Q7: LCSC C2692945 -> C53417
Changed lines of the file:
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@@
 			)
 		)
-		(property "LCSC" "C2692945"
+		(property "LCSC" "C53417"
 			(at 0 0 0)
 			(effects
@@
 			)
 		)
-		(property "LCSC" "C2692945"
+		(property "LCSC" "C53417"
 			(at 0 0 0)
 			(effects
@@
 			)
 		)
-		(property "LCSC" "C2692945"
+		(property "LCSC" "C53417"
 			(at 0 0 0)
 			(effects
@@
 			)
 		)
-		(property "LCSC" "C2692945"
+		(property "LCSC" "C53417"
 			(at 0 0 0)
 			(effects
@@
 			)
 		)
-		(property "LCSC" "C2692945"
+		(property "LCSC" "C53417"
 			(at 0 0 0)
 			(effects
@@
 			)
 		)
-		(property "LCSC" "C2692945"
+		(property "LCSC" "C53417"
 			(at 0 0 0)
 			(effects
