File: design/SBS_hw.kicad_sch (KiCad schematic)
At the start: 32 parts

Commit message: finalised, ish, will have claude review
Parts:
- added D2, D3, D4: LED, symbol Device:LED
- added R22, R23: 1k, symbol Device:R_Small
- added R24, R25, R26: 220R, symbol Device:R_Small
Connections:
- net +3.3V: now also D4.2 (A), R22.2, R23.2
- net GND: now also R24.2, R25.2, R26.2
- net MCU/LED_GREEN: now also D3.2 (A)
- net MCU/LED_RED: now also D2.2 (A)
- new net: D4.1 (K), R24.1
- new net: D3.1 (K), R26.1
- new net: D2.1 (K), R25.1
- new net BMI160/SCL: R23.1
- new net BMI160/SDA: R22.1
Other:
- added sheet BMI160 (BMI160.kicad_sch)
- sheet DRV8301 ports: added +3.3v; removed none
- sheet Power ports: added +3.3v, CURR_A, CURR_B, CURR_C, CURR_FILTER, GH_A, GH_B, GH_C, GL_A, GL_B, GL_C, GND, SH_A, SH_B, SH_C, SL_A, SL_B, SL_C, SUPPLY, TEMP; removed none
