File: design/SBS_hw.kicad_sch (KiCad schematic)
At the start: 40 parts

Commit message: Sheet 1 (SBS_hw.kicad_sch): assign footprints and part values
- LEDs D2/D3/D4: footprint LED_SMD:LED_0603_1608Metric, values LED_RED/GREEN/BLUE
- LED D?: footprint LED_SMD:LED_0603_1608Metric
- Zener D?: value BZX84C3V6, footprint Diode_SMD:D_SOT-23
- Schottky D? ×3: value 1N5819WS, footprint Diode_SMD:D_SOD-323
- USB J?: footprint Connector_USB:USB_Micro-B_Molex_105017-0001
- SERVO J?: footprint Connector_JST:JST_PH_S3B-PH-K 2mm horizontal
- HALL_ENC J?: footprint Connector_JST:JST_PH_S6B-PH-K 2mm horizontal
- COMM J?: footprint Connector_PinHeader_2.54mm 1x08
- SWD J?: footprint Connector_PinHeader_1.27mm 1x05
- CAN J?: footprint Connector_JST:JST_PH_S4B-PH-K 2mm horizontal
- Sensor Voltage JP?: footprint SolderJumper-3
- R22/R23 (1k), R24/R25/R26 (220R): footprint R_0603 HandSolder

Co-Authored-By: Claude Sonnet 4.6 <noreply@anthropic.com>
Parts:
- D2: value LED -> LED_RED; footprint (none) -> LED_SMD:LED_0603_1608Metric
- D3: value LED -> LED_GREEN; footprint (none) -> LED_SMD:LED_0603_1608Metric
- D4: value LED -> LED_BLUE; footprint (none) -> LED_SMD:LED_0603_1608Metric
- D?: footprint (none) -> LED_SMD:LED_0603_1608Metric
- D? (x3): value D_Schottky -> 1N5819WS; footprint (none) -> Diode_SMD:D_SOD-323
- D?: value D_Zener -> BZX84C3V6; footprint (none) -> Diode_SMD:D_SOT-23
- J?: footprint (none) -> Connector_USB:USB_Micro-B_Molex_105017-0001
- J?: footprint (none) -> Connector_JST:JST_PH_S3B-PH-K_1x03_P2.00mm_Horizontal
- J?: footprint (none) -> Connector_JST:JST_PH_S6B-PH-K_1x06_P2.00mm_Horizontal
- J?: footprint (none) -> Connector_PinHeader_2.54mm:PinHeader_1x08_P2.54mm_Vertical
- J?: footprint (none) -> Connector_PinHeader_1.27mm:PinHeader_1x05_P1.27mm_Vertical
- J?: footprint (none) -> Connector_JST:JST_PH_S4B-PH-K_1x04_P2.00mm_Horizontal
- JP?: footprint (none) -> Jumper:SolderJumper-3_P1.3mm_Open_SilkscreenOpenMarker_PadSize0.7x1.3mm
- R22, R23, R24, R25, R26: footprint (none) -> Resistor_SMD:R_0603_1608Metric_Pad0.98x0.95mm_HandSolder
Changed lines of the file:
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@@
 			)
 		)
-		(property "Footprint" ""
+		(property "Footprint" "Resistor_SMD:R_0603_1608Metric_Pad0.98x0.95mm_HandSolder"
 			(at 203.835 132.08 0)
 			(effects
@@
 			)
 		)
-		(property "Footprint" ""
+		(property "Footprint" "Connector_USB:USB_Micro-B_Molex_105017-0001"
 			(at 84.455 33.02 0)
 			(effects
@@
 			)
 		)
-		(property "Footprint" ""
+		(property "Footprint" "Connector_JST:JST_PH_S3B-PH-K_1x03_P2.00mm_Horizontal"
 			(at 97.79 101.6 0)
 			(effects
@@
 			)
 		)
-		(property "Footprint" ""
+		(property "Footprint" "Connector_JST:JST_PH_S6B-PH-K_1x06_P2.00mm_Horizontal"
 			(at 25.4 63.5 0)
 			(effects
@@
 			)
 		)
-		(property "Footprint" ""
+		(property "Footprint" "LED_SMD:LED_0603_1608Metric"
 			(at 99.695 184.785 0)
 			(effects
@@
 			)
 		)
-		(property "Value" "D_Schottky"
+		(property "Value" "1N5819WS"
 			(at 50.4825 88.9 0)
 			(effects
@@
 			)
 		)
-		(property "Footprint" ""
+		(property "Footprint" "Diode_SMD:D_SOD-323"
 			(at 50.8 92.71 0)
 			(effects
@@
 			)
 		)
-		(property "Footprint" ""
+		(property "Footprint" "Connector_PinHeader_2.54mm:PinHeader_1x08_P2.54mm_Vertical"
 			(at 97.79 83.82 0)
 			(effects
@@
 			)
 		)
-		(property "Value" "LED"
+		(property "Value" "LED_GREEN"
 			(at 188.595 144.145 0)
 			(effects
@@
 			)
 		)
-		(property "Footprint" ""
+		(property "Footprint" "LED_SMD:LED_0603_1608Metric"
 			(at 192.405 141.605 0)
 			(effects
@@
 			)
 		)
-		(property "Footprint" ""
+		(property "Footprint" "Connector_PinHeader_1.27mm:PinHeader_1x05_P1.27mm_Vertical"
 			(at 97.79 115.57 0)
 			(effects
@@
 			)
 		)
-		(property "Value" "D_Schottky"
+		(property "Value" "1N5819WS"
 			(at 50.4825 97.79 0)
 			(effects
@@
 			)
 		)
-		(property "Footprint" ""
+		(property "Footprint" "Diode_SMD:D_SOD-323"
 			(at 50.8 101.6 0)
 			(effects
@@
 			)
 		)
-		(property "Value" "LED"
+		(property "Value" "LED_BLUE"
 			(at 189.23 130.175 0)
 			(effects
@@
 			)
 		)
-		(property "Footprint" ""
+		(property "Footprint" "LED_SMD:LED_0603_1608Metric"
 			(at 192.405 132.08 0)
 			(effects
@@
 			)
 		)
-		(property "Footprint" ""
+		(property "Footprint" "Resistor_SMD:R_0603_1608Metric_Pad0.98x0.95mm_HandSolder"
 			(at 203.835 141.605 0)
 			(effects
@@
 			)
 		)
-		(property "Footprint" ""
+		(property "Footprint" "Resistor_SMD:R_0603_1608Metric_Pad0.98x0.95mm_HandSolder"
 			(at 192.405 111.125 0)
 			(effects
@@
 			)
 		)
-		(property "Footprint" ""
+		(property "Footprint" "Resistor_SMD:R_0603_1608Metric_Pad0.98x0.95mm_HandSolder"
 			(at 192.405 107.315 0)
 			(effects
@@
 			)
 		)
-		(property "Value" "D_Schottky"
+		(property "Value" "1N5819WS"
 			(at 64.77 107.6324 90)
 			(effects
@@
 			)
 		)
-		(property "Footprint" ""
+		(property "Footprint" "Diode_SMD:D_SOD-323"
 			(at 62.23 106.68 0)
 			(effects
@@
 			)
 		)
-		(property "Footprint" ""
+		(property "Footprint" "Connector_JST:JST_PH_S4B-PH-K_1x04_P2.00mm_Horizontal"
 			(at 97.79 48.26 0)
 			(effects
@@
 			)
 		)
-		(property "Value" "D_Zener"
+		(property "Value" "BZX84C3V6"
 			(at 26.67 114.2999 90)
 			(effects
@@
 			)
 		)
-		(property "Footprint" ""
+		(property "Footprint" "Diode_SMD:D_SOT-23"
 			(at 24.13 113.03 0)
 			(effects
@@
 			)
 		)
-		(property "Value" "LED"
+		(property "Value" "LED_RED"
 			(at 188.595 138.43 0)
 			(effects
@@
 			)
 		)
-		(property "Footprint" ""
+		(property "Footprint" "LED_SMD:LED_0603_1608Metric"
 			(at 192.405 137.16 0)
 			(effects
@@
 			)
 		)
-		(property "Footprint" ""
+		(property "Footprint" "Resistor_SMD:R_0603_1608Metric_Pad0.98x0.95mm_HandSolder"
 			(at 203.835 137.16 0)
 			(effects
@@
 			)
 		)
-		(property "Footprint" ""
+		(property "Footprint" "Jumper:SolderJumper-3_P1.3mm_Open_SilkscreenOpenMarker_PadSize0.7x1.3mm"
 			(at 40.005 31.115 0)
 			(effects

Commit message: All sheets: add LCSC part numbers to 136 components
Populated LCSC Cxxxxxx properties on every assigned component across all
6 sheets (SBS_hw, MCU, DRV8301, CAN, BMI160, Power). Remaining ~19
components (15nF/120pF 0603 caps, 2.2µF 0805, 100µF electrolytic/1210,
1k PTC, 1.27mm SWD header, solder jumper, single-pin placeholders) have
no confirmed LCSC number and are left unpopulated.

Co-Authored-By: Claude Sonnet 4.6 <noreply@anthropic.com>
Claude-Session: https://claude.ai/code/session_01DS1NowMbUxuJRBVhV127qS
Parts:
- C1, C2, C4: renamed from C?; LCSC (none) -> C14663
- C3, C5: renamed from C?; LCSC (none) -> C23630
- D1, D2, D3: renamed from D?; LCSC (none) -> C191023
- D4: renamed from D?; LCSC (none) -> C96230
- D5: renamed from D4; LCSC (none) -> C19171394
- D6: renamed from D2; LCSC (none) -> C84263
- D7: renamed from D3; LCSC (none) -> C2289
- D8: renamed from D?; LCSC (none) -> C84263
- J1: renamed from J?; LCSC (none) -> C10418
- J2: renamed from J?; LCSC (none) -> C157926
- J3: renamed from J?; LCSC (none) -> C157920
- J4: renamed from J?; LCSC (none) -> C2337
- J5: renamed from J?; LCSC (none) -> C157929
- R1: renamed from R?; LCSC (none) -> C21189
- R10: renamed from R?; LCSC (none) -> C23206
- R11: renamed from R?; LCSC (none) -> C22962
- R12: renamed from R23; LCSC (none) -> C21190
- R13: renamed from R22; LCSC (none) -> C21190
- R16: renamed from R24; LCSC (none) -> C22962
- R17: renamed from R25; LCSC (none) -> C22962
- R18: renamed from R26; LCSC (none) -> C22962
- R19: renamed from R?; LCSC (none) -> C21190
- R2, R3: renamed from R?; LCSC (none) -> C23345
- R4, R5, R6: renamed from R?; LCSC (none) -> C4190
- R7: renamed from R?; LCSC (none) -> C25804
- R8: renamed from R?; LCSC (none) -> C23153
- R9: renamed from R?; LCSC (none) -> C22775
- U1: renamed from U?; LCSC (none) -> C2151959
- gave numbers to parts that had none: 4
