File: design/BMI160.kicad_sch (KiCad schematic)
At the start: 3 parts, among them U11 BMI160

Commit message: Sheets 4–6: fix remaining blank footprints, update analog switches
CAN sheet (Sheet 4): already clean, no changes.

BMI160 sheet (Sheet 5):
- C23, C24 (2u2): footprint set to C_0603 HandSolder

Power sheet (Sheet 6):
- U8/U9/U10: Value → SN74LVC1G66DCKR, Footprint → SOT-353_SC-70-5 (MC-014 partial)
- U5/U6/U7 AD8418: Footprint → MSOP-8_3x3mm_P0.65mm
- R9/R13/R16 shunt (0.5mΩ): Footprint → R_2010_5025Metric
- J1/J2, PH_A/B/C: placeholder PinHeader_1x01 footprints
- TH1, R18-R21: R_0603 HandSolder
- C16-C22 (1n/15n/2u2): C_0603 HandSolder

Co-Authored-By: Claude Sonnet 4.6 <noreply@anthropic.com>
Parts:
- C23, C24: footprint (none) -> Capacitor_SMD:C_0603_1608Metric_Pad1.08x0.95mm_HandSolder
Changed lines of the file:
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@@
 			)
 		)
-		(property "Footprint" ""
+		(property "Footprint" "Capacitor_SMD:C_0603_1608Metric_Pad1.08x0.95mm_HandSolder"
 			(at 165.735 98.425 0)
 			(effects
@@
 			)
 		)
-		(property "Footprint" ""
+		(property "Footprint" "Capacitor_SMD:C_0603_1608Metric_Pad1.08x0.95mm_HandSolder"
 			(at 156.845 98.425 0)
 			(effects

Commit message: All sheets: add LCSC part numbers to 136 components
Populated LCSC Cxxxxxx properties on every assigned component across all
6 sheets (SBS_hw, MCU, DRV8301, CAN, BMI160, Power). Remaining ~19
components (15nF/120pF 0603 caps, 2.2µF 0805, 100µF electrolytic/1210,
1k PTC, 1.27mm SWD header, solder jumper, single-pin placeholders) have
no confirmed LCSC number and are left unpopulated.

Co-Authored-By: Claude Sonnet 4.6 <noreply@anthropic.com>
Claude-Session: https://claude.ai/code/session_01DS1NowMbUxuJRBVhV127qS
Parts:
- C59: renamed from C23; LCSC (none) -> C23630
- C60: renamed from C24; LCSC (none) -> C23630
- U15: renamed from U11; LCSC (none) -> C94021
Changed lines of the file:
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@@
 		(dnp no)
 		(fields_autoplaced yes)
-		(property "Reference" "#PWR039"
+		(property "Reference" "#PWR091"
 			(at 138.43 87.63 0)
 			(effects
@@
 			(project ""
 				(path "/dd38ec4f-50ac-4e5a-9436-c94e23afec43/b13fa9ca-c537-47cf-a098-dbc4c473d799"
-					(reference "#PWR039")
+					(reference "#PWR091")
 					(unit 1)
 				)
@@
 		(dnp no)
 		(fields_autoplaced yes)
-		(property "Reference" "#PWR040"
+		(property "Reference" "#PWR092"
 			(at 138.43 125.73 0)
 			(effects
@@
 			(project ""
 				(path "/dd38ec4f-50ac-4e5a-9436-c94e23afec43/b13fa9ca-c537-47cf-a098-dbc4c473d799"
-					(reference "#PWR040")
+					(reference "#PWR092")
 					(unit 1)
 				)
@@
 		(on_board yes)
 		(dnp no)
-		(property "Reference" "C24"
+		(property "Reference" "C60"
 			(at 168.91 97.1612 0)
 			(effects
@@
 			(project "SBS_hw"
 				(path "/dd38ec4f-50ac-4e5a-9436-c94e23afec43/b13fa9ca-c537-47cf-a098-dbc4c473d799"
-					(reference "C24")
-					(unit 1)
-				)
+					(reference "C60")
+					(unit 1)
+				)
+			)
+		)
+		(property "LCSC" "C23630"
+			(at 0 0 0)
+			(effects
+				(font
+					(size 1.27 1.27)
+				)
+				(hide yes)
 			)
 		)
@@
 		(on_board yes)
 		(dnp no)
-		(property "Reference" "C23"
+		(property "Reference" "C59"
 			(at 160.02 97.1612 0)
 			(effects
@@
 			(project ""
 				(path "/dd38ec4f-50ac-4e5a-9436-c94e23afec43/b13fa9ca-c537-47cf-a098-dbc4c473d799"
-					(reference "C23")
-					(unit 1)
-				)
+					(reference "C59")
+					(unit 1)
+				)
+			)
+		)
+		(property "LCSC" "C23630"
+			(at 0 0 0)
+			(effects
+				(font
+					(size 1.27 1.27)
+				)
+				(hide yes)
 			)
 		)
@@
 		(dnp no)
 		(fields_autoplaced yes)
-		(property "Reference" "U11"
+		(property "Reference" "U15"
 			(at 142.4783 87.63 0)
 			(effects
@@
 			(project ""
 				(path "/dd38ec4f-50ac-4e5a-9436-c94e23afec43/b13fa9ca-c537-47cf-a098-dbc4c473d799"
-					(reference "U11")
-					(unit 1)
-				)
-			)
-		)
+					(reference "U15")
+					(unit 1)
+				)
+			)
+		)
+		(property "LCSC" "C94021"
+			(at 0 0 0)
+			(effects
+				(font
+					(size 1.27 1.27)
+				)
+				(hide yes)
+			)
+		)
