File: design/CAN.kicad_sch (KiCad schematic)
At the start: 7 parts

Commit message: All sheets: add LCSC part numbers to 136 components
Populated LCSC Cxxxxxx properties on every assigned component across all
6 sheets (SBS_hw, MCU, DRV8301, CAN, BMI160, Power). Remaining ~19
components (15nF/120pF 0603 caps, 2.2µF 0805, 100µF electrolytic/1210,
1k PTC, 1.27mm SWD header, solder jumper, single-pin placeholders) have
no confirmed LCSC number and are left unpopulated.

Co-Authored-By: Claude Sonnet 4.6 <noreply@anthropic.com>
Claude-Session: https://claude.ai/code/session_01DS1NowMbUxuJRBVhV127qS
Parts:
- C39, C41: renamed from C?; LCSC (none) -> C19666
- C40, C42: renamed from C?; LCSC (none) -> C14663
- R34: renamed from R?; LCSC (none) -> C22962
- R35: renamed from R?; LCSC (none) -> C25804
- U8: renamed from U?; LCSC (none) -> C133788
Changed lines of the file:
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@@
 		(on_board yes)
 		(dnp no)
-		(property "Reference" "R?"
+		(property "Reference" "R34"
 			(at 148.59 85.09 90)
 			(effects
@@
 			(project ""
 				(path "/dd38ec4f-50ac-4e5a-9436-c94e23afec43/546412ec-fa89-4be7-b7d8-89c15693ef7f"
-					(reference "R?")
-					(unit 1)
-				)
+					(reference "R34")
+					(unit 1)
+				)
+			)
+		)
+		(property "LCSC" "C22962"
+			(at 0 0 0)
+			(effects
+				(font
+					(size 1.27 1.27)
+				)
+				(hide yes)
 			)
 		)
@@
 		(on_board yes)
 		(dnp no)
-		(property "Reference" "#PWR?"
+		(property "Reference" "#PWR068"
 			(at 123.19 80.645 0)
 			(effects
@@
 			(project ""
 				(path "/dd38ec4f-50ac-4e5a-9436-c94e23afec43/546412ec-fa89-4be7-b7d8-89c15693ef7f"
-					(reference "#PWR?")
+					(reference "#PWR068")
 					(unit 1)
 				)
@@
 		(dnp no)
 		(fields_autoplaced yes)
-		(property "Reference" "#PWR?"
+		(property "Reference" "#PWR070"
 			(at 125.73 107.315 0)
 			(effects
@@
 			(project ""
 				(path "/dd38ec4f-50ac-4e5a-9436-c94e23afec43/546412ec-fa89-4be7-b7d8-89c15693ef7f"
-					(reference "#PWR?")
+					(reference "#PWR070")
 					(unit 1)
 				)
@@
 		(on_board yes)
 		(dnp no)
-		(property "Reference" "C?"
+		(property "Reference" "C40"
 			(at 186.69 65.405 0)
 			(effects
@@
 			(project ""
 				(path "/dd38ec4f-50ac-4e5a-9436-c94e23afec43/546412ec-fa89-4be7-b7d8-89c15693ef7f"
-					(reference "C?")
-					(unit 1)
-				)
+					(reference "C40")
+					(unit 1)
+				)
+			)
+		)
+		(property "LCSC" "C14663"
+			(at 0 0 0)
+			(effects
+				(font
+					(size 1.27 1.27)
+				)
+				(hide yes)
 			)
 		)
@@
 		(on_board yes)
 		(dnp no)
-		(property "Reference" "C?"
+		(property "Reference" "C39"
 			(at 171.45 65.405 0)
 			(effects
@@
 			(project ""
 				(path "/dd38ec4f-50ac-4e5a-9436-c94e23afec43/546412ec-fa89-4be7-b7d8-89c15693ef7f"
-					(reference "C?")
-					(unit 1)
-				)
+					(reference "C39")
+					(unit 1)
+				)
+			)
+		)
+		(property "LCSC" "C19666"
+			(at 0 0 0)
+			(effects
+				(font
+					(size 1.27 1.27)
+				)
+				(hide yes)
 			)
 		)
@@
 		(on_board yes)
 		(dnp no)
-		(property "Reference" "R?"
+		(property "Reference" "R35"
 			(at 108.585 96.52 90)
 			(effects
@@
 			(project ""
 				(path "/dd38ec4f-50ac-4e5a-9436-c94e23afec43/546412ec-fa89-4be7-b7d8-89c15693ef7f"
-					(reference "R?")
-					(unit 1)
-				)
+					(reference "R35")
+					(unit 1)
+				)
+			)
+		)
+		(property "LCSC" "C25804"
+			(at 0 0 0)
+			(effects
+				(font
+					(size 1.27 1.27)
+				)
+				(hide yes)
 			)
 		)
@@
 		(on_board yes)
 		(dnp no)
-		(property "Reference" "#PWR?"
+		(property "Reference" "#PWR069"
 			(at 127 80.645 0)
 			(effects
@@
 			(project ""
 				(path "/dd38ec4f-50ac-4e5a-9436-c94e23afec43/546412ec-fa89-4be7-b7d8-89c15693ef7f"
-					(reference "#PWR?")
+					(reference "#PWR069")
 					(unit 1)
 				)
@@
 		(dnp no)
 		(fields_autoplaced yes)
-		(property "Reference" "#PWR?"
+		(property "Reference" "#PWR064"
 			(at 176.53 64.77 0)
 			(effects
@@
 			(project ""
 				(path "/dd38ec4f-50ac-4e5a-9436-c94e23afec43/546412ec-fa89-4be7-b7d8-89c15693ef7f"
-					(reference "#PWR?")
+					(reference "#PWR064")
 					(unit 1)
 				)
@@
 		(dnp no)
 		(fields_autoplaced yes)
-		(property "Reference" "#PWR?"
+		(property "Reference" "#PWR067"
 			(at 198.12 78.105 0)
 			(effects
@@
 			(project ""
 				(path "/dd38ec4f-50ac-4e5a-9436-c94e23afec43/546412ec-fa89-4be7-b7d8-89c15693ef7f"
-					(reference "#PWR?")
+					(reference "#PWR067")
 					(unit 1)
 				)
@@
 		(on_board yes)
 		(dnp no)
-		(property "Reference" "C?"
+		(property "Reference" "C42"
 			(at 208.28 65.405 0)
 			(effects
@@
 			(project ""
 				(path "/dd38ec4f-50ac-4e5a-9436-c94e23afec43/546412ec-fa89-4be7-b7d8-89c15693ef7f"
-					(reference "C?")
-					(unit 1)
-				)
+					(reference "C42")
+					(unit 1)
+				)
+			)
+		)
+		(property "LCSC" "C14663"
+			(at 0 0 0)
+			(effects
+				(font
+					(size 1.27 1.27)
+				)
+				(hide yes)
 			)
 		)
@@
 		(dnp no)
 		(fields_autoplaced yes)
-		(property "Reference" "#PWR?"
+		(property "Reference" "#PWR066"
 			(at 176.53 78.105 0)
 			(effects
@@
 			(project ""
 				(path "/dd38ec4f-50ac-4e5a-9436-c94e23afec43/546412ec-fa89-4be7-b7d8-89c15693ef7f"
-					(reference "#PWR?")
+					(reference "#PWR066")
 					(unit 1)
 				)
@@
 		(on_board yes)
 		(dnp no)
-		(property "Reference" "U?"
+		(property "Reference" "U8"
 			(at 116.205 80.01 0)
 			(effects
@@
 			(project ""
 				(path "/dd38ec4f-50ac-4e5a-9436-c94e23afec43/546412ec-fa89-4be7-b7d8-89c15693ef7f"
-					(reference "U?")
-					(unit 1)
-				)
+					(reference "U8")
+					(unit 1)
+				)
+			)
+		)
+		(property "LCSC" "C133788"
+			(at 0 0 0)
+			(effects
+				(font
+					(size 1.27 1.27)
+				)
+				(hide yes)
 			)
 		)
@@
 		(on_board yes)
 		(dnp no)
-		(property "Reference" "#PWR?"
+		(property "Reference" "#PWR065"
 			(at 198.12 64.77 0)
 			(effects
@@
 			(project ""
 				(path "/dd38ec4f-50ac-4e5a-9436-c94e23afec43/546412ec-fa89-4be7-b7d8-89c15693ef7f"
-					(reference "#PWR?")
+					(reference "#PWR065")
 					(unit 1)
 				)
@@
 		(on_board yes)
 		(dnp no)
-		(property "Reference" "C?"
+		(property "Reference" "C41"
 			(at 193.04 65.405 0)
 			(effects
@@
 			(project ""
 				(path "/dd38ec4f-50ac-4e5a-9436-c94e23afec43/546412ec-fa89-4be7-b7d8-89c15693ef7f"
-					(reference "C?")
-					(unit 1)
-				)
-			)
-		)
+					(reference "C41")
+					(unit 1)
+				)
+			)
+		)
+		(property "LCSC" "C19666"
+			(at 0 0 0)
+			(effects
+				(font
+					(size 1.27 1.27)
+				)
+				(hide yes)
+			)
+		)
