File: design/MCU.kicad_sch (KiCad schematic)
At the start: 14 parts

Commit message: Sheet 2 (MCU.kicad_sch): fix crystal; document BOOT0/PC13 and VDDA issues
Crystal Y? (MC-007 RESOLVED):
- Value: Crystal_GND24 → 8MHz
- Footprint: → Crystal:Crystal_SMD_3225-4Pin_3.2x2.5mm
  (matches LCSC C5181477 SOSET 8MHz 20pF 10ppm per BOM.md)

New issues found via direct coordinate analysis (both need KiCad wiring fixes):
- MC-013: PC13 hierarchical label placed at BOOT0 pin (y=133.35) not PC13 GPIO (y=62.23)
- MC-015: VDDA (pin 13) has no wire connection; needs +3.3V path and bypass caps

Co-Authored-By: Claude Sonnet 4.6 <noreply@anthropic.com>
Parts:
- Y?: value Crystal_GND24 -> 8MHz; footprint (none) -> Crystal:Crystal_SMD_3225-4Pin_3.2x2.5mm
Changed lines of the file:
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@@
 			)
 		)
-		(property "Value" "Crystal_GND24"
+		(property "Value" "8MHz"
 			(at 116.84 86.106 90)
 			(effects
@@
 			)
 		)
-		(property "Footprint" ""
+		(property "Footprint" "Crystal:Crystal_SMD_3225-4Pin_3.2x2.5mm"
 			(at 104.14 88.265 0)
 			(effects

Commit message: All sheets: add LCSC part numbers to 136 components
Populated LCSC Cxxxxxx properties on every assigned component across all
6 sheets (SBS_hw, MCU, DRV8301, CAN, BMI160, Power). Remaining ~19
components (15nF/120pF 0603 caps, 2.2µF 0805, 100µF electrolytic/1210,
1k PTC, 1.27mm SWD header, solder jumper, single-pin placeholders) have
no confirmed LCSC number and are left unpopulated.

Co-Authored-By: Claude Sonnet 4.6 <noreply@anthropic.com>
Claude-Session: https://claude.ai/code/session_01DS1NowMbUxuJRBVhV127qS
Parts:
- C10, C11, C13, C14, C6, C7, C8, C9: renamed from C?; LCSC (none) -> C23630
- C12: renamed from C?; LCSC (none) -> C14663
- C15, C16: renamed from C?; LCSC (none) -> C1644
- FB1: renamed from FB?; LCSC (none) -> C133937
- U2: renamed from U?; LCSC (none) -> C15742
- Y1: renamed from Y?; LCSC (none) -> C5181477
Changed lines of the file:
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@@
 		(dnp no)
 		(fields_autoplaced yes)
-		(property "Reference" "U?"
+		(property "Reference" "U2"
 			(at 160.1344 143.51 0)
 			(effects
@@
 			(project ""
 				(path "/dd38ec4f-50ac-4e5a-9436-c94e23afec43/10e71c35-5fce-44ed-b7b9-e9ee45a7ef61"
-					(reference "U?")
-					(unit 1)
-				)
+					(reference "U2")
+					(unit 1)
+				)
+			)
+		)
+		(property "LCSC" "C15742"
+			(at 0 0 0)
+			(effects
+				(font
+					(size 1.27 1.27)
+				)
+				(hide yes)
 			)
 		)
@@
 		(on_board yes)
 		(dnp no)
-		(property "Reference" "C?"
+		(property "Reference" "C8"
 			(at 118.745 40.005 0)
 			(effects
@@
 			(project ""
 				(path "/dd38ec4f-50ac-4e5a-9436-c94e23afec43/10e71c35-5fce-44ed-b7b9-e9ee45a7ef61"
-					(reference "C?")
-					(unit 1)
-				)
+					(reference "C8")
+					(unit 1)
+				)
+			)
+		)
+		(property "LCSC" "C23630"
+			(at 0 0 0)
+			(effects
+				(font
+					(size 1.27 1.27)
+				)
+				(hide yes)
 			)
 		)
@@
 		(on_board yes)
 		(dnp no)
-		(property "Reference" "C?"
+		(property "Reference" "C15"
 			(at 87.63 82.55 0)
 			(effects
@@
 			(project ""
 				(path "/dd38ec4f-50ac-4e5a-9436-c94e23afec43/10e71c35-5fce-44ed-b7b9-e9ee45a7ef61"
-					(reference "C?")
-					(unit 1)
-				)
+					(reference "C15")
+					(unit 1)
+				)
+			)
+		)
+		(property "LCSC" "C1644"
+			(at 0 0 0)
+			(effects
+				(font
+					(size 1.27 1.27)
+				)
+				(hide yes)
 			)
 		)
@@
 		(dnp no)
 		(fields_autoplaced yes)
-		(property "Reference" "#PWR?"
+		(property "Reference" "#PWR034"
 			(at 154.305 156.845 0)
 			(effects
@@
 			(project ""
 				(path "/dd38ec4f-50ac-4e5a-9436-c94e23afec43/10e71c35-5fce-44ed-b7b9-e9ee45a7ef61"
-					(reference "#PWR?")
+					(reference "#PWR034")
 					(unit 1)
 				)
@@
 		(on_board yes)
 		(dnp no)
-		(property "Reference" "C?"
+		(property "Reference" "C12"
 			(at 119.38 58.42 0)
 			(effects
@@
 			(project ""
 				(path "/dd38ec4f-50ac-4e5a-9436-c94e23afec43/10e71c35-5fce-44ed-b7b9-e9ee45a7ef61"
-					(reference "C?")
-					(unit 1)
-				)
+					(reference "C12")
+					(unit 1)
+				)
+			)
+		)
+		(property "LCSC" "C14663"
+			(at 0 0 0)
+			(effects
+				(font
+					(size 1.27 1.27)
+				)
+				(hide yes)
 			)
 		)
@@
 		(on_board yes)
 		(dnp no)
-		(property "Reference" "#PWR?"
+		(property "Reference" "#PWR032"
 			(at 130.81 85.09 0)
 			(effects
@@
 			(project ""
 				(path "/dd38ec4f-50ac-4e5a-9436-c94e23afec43/10e71c35-5fce-44ed-b7b9-e9ee45a7ef61"
-					(reference "#PWR?")
+					(reference "#PWR032")
 					(unit 1)
 				)
@@
 		(on_board yes)
 		(dnp no)
-		(property "Reference" "C?"
+		(property "Reference" "C6"
 			(at 167.64 39.37 0)
 			(effects
@@
 			(project ""
 				(path "/dd38ec4f-50ac-4e5a-9436-c94e23afec43/10e71c35-5fce-44ed-b7b9-e9ee45a7ef61"
-					(reference "C?")
-					(unit 1)
-				)
+					(reference "C6")
+					(unit 1)
+				)
+			)
+		)
+		(property "LCSC" "C23630"
+			(at 0 0 0)
+			(effects
+				(font
+					(size 1.27 1.27)
+				)
+				(hide yes)
 			)
 		)
@@
 		(on_board yes)
 		(dnp no)
-		(property "Reference" "#PWR?"
+		(property "Reference" "#PWR029"
 			(at 133.35 54.61 0)
 			(effects
@@
 			(project ""
 				(path "/dd38ec4f-50ac-4e5a-9436-c94e23afec43/10e71c35-5fce-44ed-b7b9-e9ee45a7ef61"
-					(reference "#PWR?")
+					(reference "#PWR029")
 					(unit 1)
 				)
@@
 		(on_board yes)
 		(dnp no)
-		(property "Reference" "#PWR?"
+		(property "Reference" "#PWR030"
 			(at 174.625 54.61 0)
 			(effects
@@
 			(project ""
 				(path "/dd38ec4f-50ac-4e5a-9436-c94e23afec43/10e71c35-5fce-44ed-b7b9-e9ee45a7ef61"
-					(reference "#PWR?")
+					(reference "#PWR030")
 					(unit 1)
 				)
@@
 		(on_board yes)
 		(dnp no)
-		(property "Reference" "C?"
+		(property "Reference" "C7"
 			(at 181.61 39.37 0)
 			(effects
@@
 			(project ""
 				(path "/dd38ec4f-50ac-4e5a-9436-c94e23afec43/10e71c35-5fce-44ed-b7b9-e9ee45a7ef61"
-					(reference "C?")
-					(unit 1)
-				)
+					(reference "C7")
+					(unit 1)
+				)
+			)
+		)
+		(property "LCSC" "C23630"
+			(at 0 0 0)
+			(effects
+				(font
+					(size 1.27 1.27)
+				)
+				(hide yes)
 			)
 		)
@@
 		(on_board yes)
 		(dnp no)
-		(property "Reference" "#PWR?"
+		(property "Reference" "#PWR033"
 			(at 98.425 103.505 0)
 			(effects
@@
 			(project ""
 				(path "/dd38ec4f-50ac-4e5a-9436-c94e23afec43/10e71c35-5fce-44ed-b7b9-e9ee45a7ef61"
-					(reference "#PWR?")
+					(reference "#PWR033")
 					(unit 1)
 				)
@@
 		(on_board yes)
 		(dnp no)
-		(property "Reference" "FB?"
+		(property "Reference" "FB1"
 			(at 163.83 37.465 0)
 			(effects
@@
 			(project ""
 				(path "/dd38ec4f-50ac-4e5a-9436-c94e23afec43/10e71c35-5fce-44ed-b7b9-e9ee45a7ef61"
-					(reference "FB?")
-					(unit 1)
-				)
+					(reference "FB1")
+					(unit 1)
+				)
+			)
+		)
+		(property "LCSC" "C133937"
+			(at 0 0 0)
+			(effects
+				(font
+					(size 1.27 1.27)
+				)
+				(hide yes)
 			)
 		)
@@
 		(dnp no)
 		(fields_autoplaced yes)
-		(property "Reference" "Y?"
+		(property "Reference" "Y1"
 			(at 116.84 83.566 90)
 			(effects
@@
 			(project ""
 				(path "/dd38ec4f-50ac-4e5a-9436-c94e23afec43/10e71c35-5fce-44ed-b7b9-e9ee45a7ef61"
-					(reference "Y?")
-					(unit 1)
-				)
+					(reference "Y1")
+					(unit 1)
+				)
+			)
+		)
+		(property "LCSC" "C5181477"
+			(at 0 0 0)
+			(effects
+				(font
+					(size 1.27 1.27)
+				)
+				(hide yes)
 			)
 		)
@@
 		(on_board yes)
 		(dnp no)
-		(property "Reference" "C?"
+		(property "Reference" "C13"
 			(at 123.825 72.39 0)
 			(effects
@@
 			(project ""
 				(path "/dd38ec4f-50ac-4e5a-9436-c94e23afec43/10e71c35-5fce-44ed-b7b9-e9ee45a7ef61"
-					(reference "C?")
-					(unit 1)
-				)
+					(reference "C13")
+					(unit 1)
+				)
+			)
+		)
+		(property "LCSC" "C23630"
+			(at 0 0 0)
+			(effects
+				(font
+					(size 1.27 1.27)
+				)
+				(hide yes)
 			)
 		)
@@
 		(on_board yes)
 		(dnp no)
-		(property "Reference" "C?"
+		(property "Reference" "C16"
 			(at 87.63 90.805 0)
 			(effects
@@
 			(project ""
 				(path "/dd38ec4f-50ac-4e5a-9436-c94e23afec43/10e71c35-5fce-44ed-b7b9-e9ee45a7ef61"
-					(reference "C?")
-					(unit 1)
-				)
+					(reference "C16")
+					(unit 1)
+				)
+			)
+		)
+		(property "LCSC" "C1644"
+			(at 0 0 0)
+			(effects
+				(font
+					(size 1.27 1.27)
+				)
+				(hide yes)
 			)
 		)
@@
 		(on_board yes)
 		(dnp no)
-		(property "Reference" "#PWR?"
+		(property "Reference" "#PWR031"
 			(at 124.46 69.85 0)
 			(effects
@@
 			(project ""
 				(path "/dd38ec4f-50ac-4e5a-9436-c94e23afec43/10e71c35-5fce-44ed-b7b9-e9ee45a7ef61"
-					(reference "#PWR?")
+					(reference "#PWR031")
 					(unit 1)
 				)
@@
 		(on_board yes)
 		(dnp no)
-		(property "Reference" "C?"
+		(property "Reference" "C14"
 			(at 137.795 72.39 0)
 			(effects
@@
 			(project ""
 				(path "/dd38ec4f-50ac-4e5a-9436-c94e23afec43/10e71c35-5fce-44ed-b7b9-e9ee45a7ef61"
-					(reference "C?")
-					(unit 1)
-				)
+					(reference "C14")
+					(unit 1)
+				)
+			)
+		)
+		(property "LCSC" "C23630"
+			(at 0 0 0)
+			(effects
+				(font
+					(size 1.27 1.27)
+				)
+				(hide yes)
 			)
 		)
@@
 		(on_board yes)
 		(dnp no)
-		(property "Reference" "C?"
+		(property "Reference" "C9"
 			(at 132.715 40.005 0)
 			(effects
@@
 			(project ""
 				(path "/dd38ec4f-50ac-4e5a-9436-c94e23afec43/10e71c35-5fce-44ed-b7b9-e9ee45a7ef61"
-					(reference "C?")
-					(unit 1)
-				)
+					(reference "C9")
+					(unit 1)
+				)
+			)
+		)
+		(property "LCSC" "C23630"
+			(at 0 0 0)
+			(effects
+				(font
+					(size 1.27 1.27)
+				)
+				(hide yes)
 			)
 		)
@@
 		(on_board yes)
 		(dnp no)
-		(property "Reference" "C?"
+		(property "Reference" "C11"
 			(at 149.225 40.005 0)
 			(effects
@@
 			(project ""
 				(path "/dd38ec4f-50ac-4e5a-9436-c94e23afec43/10e71c35-5fce-44ed-b7b9-e9ee45a7ef61"
-					(reference "C?")
-					(unit 1)
-				)
+					(reference "C11")
+					(unit 1)
+				)
+			)
+		)
+		(property "LCSC" "C23630"
+			(at 0 0 0)
+			(effects
+				(font
+					(size 1.27 1.27)
+				)
+				(hide yes)
 			)
 		)
@@
 		(on_board yes)
 		(dnp no)
-		(property "Reference" "C?"
+		(property "Reference" "C10"
 			(at 135.255 40.005 0)
 			(effects
@@
 			(project ""
 				(path "/dd38ec4f-50ac-4e5a-9436-c94e23afec43/10e71c35-5fce-44ed-b7b9-e9ee45a7ef61"
-					(reference "C?")
-					(unit 1)
-				)
-			)
-		)
+					(reference "C10")
+					(unit 1)
+				)
+			)
+		)
+		(property "LCSC" "C23630"
+			(at 0 0 0)
+			(effects
+				(font
+					(size 1.27 1.27)
+				)
+				(hide yes)
+			)
+		)
